Commit message: feature:修改kr10包

File: kr10/urdf/kr10.urdf (robot description, URDF)
Before this commit: robot kr10, 8 links, 7 joints
Links:
- removed link dummy
- link link1: mass 6.76282099629239 -> 6.2751497959128
- link link2: mass 11.0807759235315 -> 10.0623910575082
- link link3: mass 2.87413726622841 -> 2.87413726622842
- link link4: mass 4.03616260529762 -> 4.03623874477417
- link link5: mass 0.442068337293596 -> 0.4420683299725
- link link6: mass 0.822898961680664 -> 0.213549096503453
Joints:
- removed joint dummy_joint
- joint joint1: limit (none) -> lower=-3 upper=3 effort=0 velocity=0; type continuous -> revolute
- joint joint2: limit (none) -> lower=-1.4 upper=2.1 effort=0 velocity=0; type continuous -> revolute
- joint joint3: limit (none) -> lower=-4 upper=1 effort=0 velocity=0; origin xyz=0.29844 -0.47385 0.0035 rpy=3.1416 0 1.5708 -> xyz=0.25768 -0.49719 0.0035 rpy=-3.1416 0 1.5708; type continuous -> revolute
- joint joint5: limit (none) -> lower=-1.8 upper=2.1 effort=0 velocity=0; origin xyz=3.2873E-05 0.00024783 0.398 rpy=1.5708 -0.94181 -0.13187 -> xyz=9.6051E-05 0.00023081 0.398 rpy=1.5708 -0.97526 -0.39435; type continuous -> revolute
- joint joint6: origin xyz=0.034487 0.056858 0.00025 rpy=-1.5708 0.091019 -0.54522 -> xyz=0.050858 0.042845 0.00025 rpy=-1.5708 0.34761 -0.87071

File: kr10/urdf/kr10.xacro (robot description, xacro)
@@ -57,5 +57,5 @@
         ixz="0.0056899080162169"
         iyy="0.13962559834333"
-        iyz="-8.42142079241257E-06"
+        iyz="-8.4214207924127E-06"
         izz="0.121027155275122" />
     </inertial>
@@ -88,15 +88,15 @@
     <inertial>
       <origin
-        xyz="0.0040119831576042 0.0153784833152217 0.115002757128672"
-        rpy="0 0 0" />
-      <mass
-        value="6.76282099629239" />
-      <inertia
-        ixx="0.0884793533754446"
-        ixy="0.00833284746456488"
-        ixz="-0.00550868593247773"
-        iyy="0.0541081305599748"
-        iyz="-0.000877214595804581"
-        izz="0.070648702343058" />
+        xyz="0.00741380480149578 0.00354552947139167 0.115715412511507"
+        rpy="0 0 0" />
+      <mass
+        value="6.2751497959128" />
+      <inertia
+        ixx="0.0751893674671946"
+        ixy="0.00504886489144856"
+        ixz="-0.00509592816750828"
+        iyy="0.0510924965053144"
+        iyz="-0.001549309062334"
+        izz="0.0562677349522946" />
     </inertial>
     <visual>
@@ -126,5 +126,5 @@
   <joint
     name="joint1"
-    type="continuous">
+    type="revolute">
     <origin
       xyz="0 0 0.217"
@@ -136,4 +136,9 @@
     <axis
       xyz="0 0 1" />
+    <limit
+      lower="-3"
+      upper="3"
+      effort="0"
+      velocity="0" />
   </joint>
   <link
@@ -141,15 +146,15 @@
     <inertial>
       <origin
-        xyz="0.140846409337324 -0.23465945327983 0.0150230251076055"
-        rpy="0 0 0" />
-      <mass
-        value="11.0807759235315" />
-      <inertia
-        ixx="0.413654939941552"
-        ixy="0.222046654839175"
-        ixz="-0.0120209374122503"
-        iyy="0.217225182156573"
-        iyz="0.013548271985692"
-        izz="0.516035383833047" />
+        xyz="0.112673325433516 -0.235533330268791 5.25939883689319E-05"
+        rpy="0 0 0" />
+      <mass
+        value="10.0623910575082" />
+      <inertia
+        ixx="0.373446746946084"
+        ixy="0.169218239470221"
+        ixz="-0.000352160811815804"
+        iyy="0.131793291732547"
+        iyz="0.000952442844566425"
+        izz="0.442938494752101" />
     </inertial>
     <visual>
@@ -179,5 +184,5 @@
   <joint
     name="joint2"
-    type="continuous">
+    type="revolute">
     <origin
       xyz="0.025397 0.00050592 0.183"
@@ -189,4 +194,9 @@
     <axis
       xyz="0 0 -1" />
+    <limit
+      lower="-1.4"
+      upper="2.1"
+      effort="0"
+      velocity="0" />
   </joint>
   <link
@@ -194,15 +204,15 @@
     <inertial>
       <origin
-        xyz="0.000529908025402204 0.019176079655101 -2.46422129662194E-05"
-        rpy="0 0 0" />
-      <mass
-        value="2.87413726622841" />
-      <inertia
-        ixx="0.0106153706452693"
-        ixy="-0.000284572592443034"
-        ixz="-3.57139634988392E-06"
-        iyy="0.00740315810462332"
-        iyz="1.82140206131432E-06"
-        izz="0.0111376816178896" />
+        xyz="0.000529908025397541 0.0191760796551027 -2.4642212648307E-05"
+        rpy="0 0 0" />
+      <mass
+        value="2.87413726622842" />
+      <inertia
+        ixx="0.0106153706452702"
+        ixy="-0.000284572592443065"
+        ixz="-3.571396350265E-06"
+        iyy="0.00740315810462365"
+        iyz="1.82140206105029E-06"
+        izz="0.0111376816178918" />
     </inertial>
     <visual>
@@ -232,8 +242,8 @@
   <joint
     name="joint3"
-    type="continuous">
-    <origin
-      xyz="0.29844 -0.47385 0.0035"
-      rpy="3.1416 0 1.5708" />
+    type="revolute">
+    <origin
+      xyz="0.25768 -0.49719 0.0035"
+      rpy="-3.1416 0 1.5708" />
     <parent
       link="link2" />
@@ -242,4 +252,9 @@
     <axis
       xyz="0 0 -1" />
+    <limit
+      lower="-4"
+      upper="1"
+      effort="0"
+      velocity="0" />
   </joint>
   <link
@@ -247,15 +262,15 @@
     <inertial>
       <origin
-        xyz="0.000393134931056194 0.000448210661311177 0.185101232919221"
-        rpy="0 0 0" />
-      <mass
-        value="4.03616260529762" />
-      <inertia
-        ixx="0.0515994204320357"
-        ixy="-0.000136107202626716"
-        ixz="-1.47461819117842E-05"
-        iyy="0.05068879924868"
-        iyz="-0.000237044049748255"
-        izz="0.0073432735506533" />
+        xyz="0.000495827295870943 0.000331263303056328 0.185104333291848"
+        rpy="0 0 0" />
+      <mass
+        value="4.03623874477417" />
+      <inertia
+        ixx="0.0514724229213813"
+        ixy="-0.000345898984168441"
+        ixz="-7.55534798658624E-05"
+        iyy="0.0508207618372116"
+        iyz="-0.000225438428481011"
+        izz="0.00734338590437416" />
     </inertial>
     <visual>
@@ -300,15 +315,15 @@
     <inertial>
       <origin
-        xyz="0.00816244459630874 0.0135157135600389 0.00216370086017081"
-        rpy="0 0 0" />
-      <mass
-        value="0.442068337293596" />
-      <inertia
-        ixx="0.000496980230553028"
-        ixy="-0.00010798453757304"
-        ixz="8.90106783261052E-06"
-        iyy="0.000383724805144781"
-        iyz="1.40522567079195E-05"
-        izz="0.000528480900593434" />
+        xyz="0.0120557743377237 0.0101959936253579 0.0021636985615841"
+        rpy="0 0 0" />
+      <mass
+        value="0.4420683299725" />
+      <inertia
+        ixx="0.000419965604922443"
+        ixy="-0.000120215358737915"
+        ixz="1.29271922535509E-05"
+        iyy="0.00046073941946462"
+        iyz="1.04681508421518E-05"
+        izz="0.000528480867675673" />
     </inertial>
     <visual>
@@ -338,8 +353,8 @@
   <joint
     name="joint5"
-    type="continuous">
-    <origin
-      xyz="3.2873E-05 0.00024783 0.398"
-      rpy="1.5708 -0.94181 -0.13187" />
+    type="revolute">
+    <origin
+      xyz="9.6051E-05 0.00023081 0.398"
+      rpy="1.5708 -0.97526 -0.39435" />
     <parent
       link="link4" />
@@ -348,4 +363,9 @@
     <axis
       xyz="0 0 -1" />
+    <limit
+      lower="-1.8"
+      upper="2.1"
+      effort="0"
+      velocity="0" />
   </joint>
   <link
@@ -353,15 +373,15 @@
     <inertial>
       <origin
-        xyz="7.16188552929431E-06 2.08076229788468E-05 0.0636648540462599"
-        rpy="0 0 0" />
-      <mass
-        value="0.822898961680664" />
-      <inertia
-        ixx="0.00125117967087411"
-        ixy="6.51863943772484E-09"
-        ixz="1.71586483774342E-07"
-        iyy="0.00125119624163199"
-        iyz="5.20683250245256E-07"
-        izz="0.000989806183652223" />
+        xyz="-2.27839703337285E-06 -1.67395761618838E-06 0.0553153630699634"
+        rpy="0 0 0" />
+      <mass
+        value="0.213549096503453" />
+      <inertia
+        ixx="0.000219860024372743"
+        ixy="-4.50770251278094E-09"
+        ixz="-2.33140665193661E-08"
+        iyy="0.000219862847887346"
+        iyz="-1.71290426984171E-08"
+        izz="7.43113458858691E-05" />
     </inertial>
     <visual>
@@ -393,6 +413,6 @@
     type="continuous">
     <origin
-      xyz="0.034487 0.056858 0.00025"
-      rpy="-1.5708 0.091019 -0.54522" />
+      xyz="0.050858 0.042845 0.00025"
+      rpy="-1.5708 0.34761 -0.87071" />
     <parent
       link="link5" />
