Commit message: fixbug:修复gazebo中机械臂解体bug

File: kr10/urdf/kr10.xacro (robot description, xacro)
@@ -41,5 +41,5 @@
             </geometry>
         </collision>
-        <!-- <xacro:inertial_matrix mass="500"/> -->
+        <xacro:inertial_matrix mass="500"/>
     </link>
   <!-- /////////////////////////////////////   BASE LINK    ////////////////////////////////////////////// -->
@@ -139,6 +139,7 @@
       lower="-3"
       upper="3"
-      effort="0"
-      velocity="0" />
+        effort="300"
+        velocity="1" />
+      <dynamics damping="10.0" friction="0.0"/>
   </joint>
   <link
@@ -197,6 +198,7 @@
       lower="-1.4"
       upper="2.1"
-      effort="0"
-      velocity="0" />
+      effort="300"
+      velocity="1" />
+    <dynamics damping="10" friction="0.0"/>
   </joint>
   <link
@@ -255,6 +257,7 @@
       lower="-4"
       upper="1"
-      effort="0"
-      velocity="0" />
+      effort="300"
+      velocity="1" />
+    <dynamics damping="10" friction="0.0"/>
   </joint>
   <link
@@ -310,4 +313,5 @@
     <axis
       xyz="0 0 -1" />
+    <dynamics damping="5" friction="0.0"/>
   </joint>
   <link
@@ -366,6 +370,7 @@
       lower="-1.8"
       upper="2.1"
-      effort="0"
-      velocity="0" />
+      effort="300"
+      velocity="1" />
+    <dynamics damping="1" friction="0.0"/>
   </joint>
   <link
@@ -421,4 +426,5 @@
     <axis
       xyz="0 0 1" />
+    <dynamics damping="1" friction="0.0"/>
   </joint>
     <!-- /////////////////////////////////   Gazebo   ////////////////////////////////////// -->

File: kr160/urdf/kr10.xacro (robot description, xacro)
@@ -97,6 +97,7 @@
       lower="-3"
       upper="3"
-      effort="0"
-      velocity="0" />
+          effort="300"
+          velocity="1" />
+        <dynamics damping="10.0" friction="0.0"/>
   </joint>
   <link
@@ -155,6 +156,7 @@
       lower="-1.4"
       upper="2.1"
-      effort="0"
-      velocity="0" />
+      effort="300"
+      velocity="1" />
+    <dynamics damping="10" friction="0.0"/>
   </joint>
   <link
@@ -213,6 +215,7 @@
       lower="-4"
       upper="1"
-      effort="0"
-      velocity="0" />
+      effort="300"
+      velocity="1" />
+    <dynamics damping="10" friction="0.0"/>
   </joint>
   <link
@@ -268,4 +271,5 @@
     <axis
       xyz="0 0 -1" />
+    <dynamics damping="5" friction="0.0"/>
   </joint>
   <link
@@ -324,6 +328,7 @@
       lower="-1.8"
       upper="2.1"
-      effort="0"
-      velocity="0" />
+      effort="300"
+      velocity="1" />
+    <dynamics damping="1" friction="0.0"/>
   </joint>
   <link
@@ -379,4 +384,5 @@
     <axis
       xyz="0 0 1" />
+    <dynamics damping="1" friction="0.0"/>
   </joint>
   </xacro:macro>

File: kr160/urdf/kr60.xacro (robot description, xacro)
@@ -97,6 +97,7 @@
       lower="-3.14"
       upper="3.14"
-      effort="0"
-      velocity="0" />
+      effort="300"
+      velocity="1" />
+    <dynamics damping="50.0" friction="0.0"/>
   </joint>
   <link
@@ -155,6 +156,7 @@
       lower="-1.2"
       upper="1.4"
-      effort="0"
-      velocity="0" />
+      effort="300"
+      velocity="1" />
+    <dynamics damping="20.0" friction="0.0"/>
   </joint>
   <link
@@ -213,6 +215,7 @@
       lower="-4"
       upper="1.1"
-      effort="0"
-      velocity="0" />
+      effort="300"
+      velocity="1" />
+    <dynamics damping="10.0" friction="0.0"/>
   </joint>
   <link
@@ -271,6 +274,7 @@
       lower="-3.14"
       upper="3.14"
-      effort="0"
-      velocity="0" />
+      effort="300"
+      velocity="1" />
+    <dynamics damping="10.0" friction="0.0"/>
   </joint>
   <link
@@ -329,6 +333,7 @@
       lower="-3.2"
       upper="1.52"
-      effort="0"
-      velocity="0" />
+      effort="300"
+      velocity="1" />
+    <dynamics damping="5.0" friction="0.0"/>
   </joint>
   <link
@@ -387,6 +392,7 @@
       lower="-3.14"
       upper="3.14"
-      effort="0"
-      velocity="0" />
+      effort="300"
+      velocity="1" />
+    <dynamics damping="1.0" friction="0.0"/>
   </joint>
   <!-- //////////////////////////////////////   finger   ////////////////////////////////////////////// -->
@@ -446,6 +452,7 @@
       lower="-1"
       upper="0.2"
-      effort="0"
-      velocity="0" />
+      effort="300"
+      velocity="1" />
+    <dynamics damping="1.0" friction="0.0"/>
   </joint>
   <link
@@ -504,6 +511,7 @@
       lower="-1"
       upper="0.2"
-      effort="0"
-      velocity="0" />
+      effort="300"
+      velocity="1" />
+    <dynamics damping="1.0" friction="0.0"/>
   </joint>
     <!-- Grasping frame -->

File: kr60/urdf/kr60.xacro (robot description, xacro)
@@ -139,6 +139,7 @@
       lower="-3.14"
       upper="3.14"
-      effort="0"
-      velocity="0" />
+      effort="300"
+      velocity="1" />
+    <dynamics damping="50.0" friction="0.0"/>
   </joint>
   <link
@@ -197,6 +198,7 @@
       lower="-1.2"
       upper="1.4"
-      effort="0"
-      velocity="0" />
+      effort="300"
+      velocity="1" />
+    <dynamics damping="20.0" friction="0.0"/>
   </joint>
   <link
@@ -255,6 +257,7 @@
       lower="-4"
       upper="1.1"
-      effort="0"
-      velocity="0" />
+      effort="300"
+      velocity="1" />
+    <dynamics damping="10.0" friction="0.0"/>
   </joint>
   <link
@@ -313,6 +316,7 @@
       lower="-3.14"
       upper="3.14"
-      effort="0"
-      velocity="0" />
+      effort="300"
+      velocity="1" />
+    <dynamics damping="10.0" friction="0.0"/>
   </joint>
   <link
@@ -371,6 +375,7 @@
       lower="-3.2"
       upper="1.52"
-      effort="0"
-      velocity="0" />
+      effort="300"
+      velocity="1" />
+    <dynamics damping="5.0" friction="0.0"/>
   </joint>
   <link
@@ -429,6 +434,7 @@
       lower="-3.14"
       upper="3.14"
-      effort="0"
-      velocity="0" />
+      effort="300"
+      velocity="1" />
+    <dynamics damping="1.0" friction="0.0"/>
   </joint>
   <!-- //////////////////////////////////////   finger   ////////////////////////////////////////////// -->
@@ -488,6 +494,7 @@
       lower="-1"
       upper="0.2"
-      effort="0"
-      velocity="0" />
+      effort="300"
+      velocity="1" />
+    <dynamics damping="1.0" friction="0.0"/>
   </joint>
   <link
@@ -546,6 +553,7 @@
       lower="-1"
       upper="0.2"
-      effort="0"
-      velocity="0" />
+      effort="300"
+      velocity="1" />
+    <dynamics damping="1.0" friction="0.0"/>
   </joint>
     <!-- Grasping frame -->
