Commit message: feature:增加kr160_moveit_config；bugfix:修复kr160 urdf bug

File: kr160/urdf/kr160.xacro (robot description, xacro)
@@ -28,5 +28,5 @@
             <origin xyz=" 0 0 -0.02"  rpy="0 0 0"/>
                 <geometry>
-                      <box size="1 1 0.02" />
+                      <box size="5 1 0.02" />
                 </geometry>
             <material name="Brown" />
@@ -35,5 +35,5 @@
           <origin xyz=" 0 0 -0.02"  rpy="0 0 0"/>
           <geometry>
-              <box size="1 1 0.02" />
+              <box size="5 1 0.02" />
           </geometry>
       </collision>
@@ -41,7 +41,7 @@
   </link>
   <!-- /////////////////////////////////   kr10   ////////////////////////////////////// -->
-  <xacro:kr10 prefix="kr10" base_parent="dummy"/>
+  <xacro:kr10 prefix="kr10"/>
   <joint name="dummy_joint_kr10" type="fixed">
-    <origin xyz="0 0 0" rpy="0 0 0" />
+    <origin xyz="-1.5 0 0" rpy="0 0 0" />
     <parent link="dummy"/>
     <child link="kr10_base_link"/>
@@ -50,5 +50,5 @@
   <xacro:kr60 prefix="kr60"/>
   <joint name="dummy_joint_kr60" type="fixed">
-    <origin xyz="0 0 0" rpy="0 0 0" />
+    <origin xyz="1.5 0 0" rpy="0 0 3.14" />
     <parent link="dummy"/>
     <child link="kr60_base_link"/>
@@ -68,19 +68,31 @@
         </transmission>
     </xacro:macro>
-    <xacro:transmission_block joint_name="joint1"/>
-    <xacro:transmission_block joint_name="joint2"/>
-    <xacro:transmission_block joint_name="joint3"/>
-    <xacro:transmission_block joint_name="joint4"/>
-    <xacro:transmission_block joint_name="joint5"/>
-    <xacro:transmission_block joint_name="joint6"/>
-    <xacro:transmission_block joint_name="finger_joint1"/>
-    <xacro:transmission_block joint_name="finger_joint2"/>
+    <xacro:transmission_block joint_name="kr10_joint1"/>
+    <xacro:transmission_block joint_name="kr10_joint2"/>
+    <xacro:transmission_block joint_name="kr10_joint3"/>
+    <xacro:transmission_block joint_name="kr10_joint4"/>
+    <xacro:transmission_block joint_name="kr10_joint5"/>
+    <xacro:transmission_block joint_name="kr10_joint6"/>
+    <xacro:transmission_block joint_name="kr60_joint1"/>
+    <xacro:transmission_block joint_name="kr60_joint2"/>
+    <xacro:transmission_block joint_name="kr60_joint3"/>
+    <xacro:transmission_block joint_name="kr60_joint4"/>
+    <xacro:transmission_block joint_name="kr60_joint5"/>
+    <xacro:transmission_block joint_name="kr60_joint6"/>
+    <xacro:transmission_block joint_name="kr60_finger_joint1"/>
+    <xacro:transmission_block joint_name="kr60_finger_joint2"/>
     <!-- ros_control plugin -->
     <gazebo>
         <plugin name="gazebo_ros_control" filename="libgazebo_ros_control.so">
-            <robotNamespace>/kr60</robotNamespace>
+            <robotNamespace>/kr160</robotNamespace>
             <robotSimType>gazebo_ros_control/DefaultRobotHWSim</robotSimType>
             <legacyModeNS>true</legacyModeNS>
         </plugin>
     </gazebo>
+    <!-- default joint position -->
+    <!-- kr10: -0.17 0.28 -0.55 0.00 -1.35 -0.01 -->
+    <!-- kr60: -0.21 0.38 0.01 0.09 -2.35 0.00 0.00 0.00 -->
+    <!-- cylinders -->
+    <!-- cylinder0: 0.1 0.05-->
+    <!-- cylinder1: 0.15 0.3 -->
 </robot>

File: kr160/urdf/kr60.xacro (robot description, xacro)
@@ -1,5 +1,5 @@
 <?xml version="1.0"?>
 <robot name="kr60" xmlns:xacro="http://ros.org/wiki/xacro">
-  <xacro:macro name="kr60" param="prefix:=kr60">
+  <xacro:macro name="kr60" params="prefix:=kr60">
   <link
     name="${prefix}_base_link">
